Commit message: Add documentaiton
Signed-off-by: Christoph Hellmann Santos <christoph.hellmann.santos@ipa.fraunhofer.de>

File: urdf/robby.robot.xacro (robot description, xacro)
@@ -39,5 +39,5 @@
         <parent link="${prefix}base_link"/>
         <child link="${prefix}left_wheel_link"/>
-        <origin xyz="-0.05 0.08 0.021" rpy="1.57 0 0"/>
+        <origin xyz="-0.05 0.12 0.021" rpy="1.57 0 0"/>
         <axis xyz="0 0 -1" />
     </joint>
@@ -45,5 +45,5 @@
         <parent link="${prefix}base_link"/>
         <child link="${prefix}right_wheel_link"/>
-        <origin xyz="-0.05 -0.080 0.021" rpy="-1.57 0 0"/>
+        <origin xyz="-0.05 -0.12 0.021" rpy="-1.57 0 0"/>
         <axis xyz="0 0 1" />
     </joint>
